File: VGA_Zero.kicad_pcb (KiCad board)
At the start: 2 copper layers, 65 x 30 mm, 33 parts, among them J1 VGA, J19 BARREL_JACK, J2 CONN_02X20, J3 AUDIO, J4 SPI

Commit message: rev2
Parts:
- moved J5 1.52 mm to (31.0, 30.0)
- moved J1 1.50 mm to (62.5, 20.0)
- moved J3 0.70 mm to (41.0, 20.0)
- renumbered J19 to J5
Routing:
- net GND: track 105.4 -> 121.2 mm, vias 1 -> 2
- net /VGAB: track 19.2 -> 18.1 mm
- net /VGAG: track 16.3 -> 15.2 mm
- net /VGAR: track 18.3 -> 17.2 mm
- net Net-(C4-Pad2): track 14.0 -> 14.9 mm
- net /VGAH: track 33.6 -> 34.3 mm
- net Net-(C2-Pad2): track 25.5 -> 25.0 mm
- net /VGAV: track 25.4 -> 26.0 mm
Other:
- board text added: "Desingned by Laurent Le Goff (2017) http://github.com/llegoff/VGA_Zero Use dtoverlay dpi24 with parameter dpi_output_format=0x13 For Audio & SPI, remake dpi24.dtbo without pin GPIO 9 10 11 18 19 25 26 27 dtoverlay=pwm-2chan,pin=18,func=2,pin2=19,func2=2"
- board text removed: "Desingned by Laurent Le Goff (2017) Use dtoverlay dpi24 with parameter dpi_output_format=0x13 For Audio & SPI, remake dpi24.dtbo without pin GPIO 9 10 11 18 19 25 26 27 dtoverlay=pwm-2chan,pin=18,func=2,pin2=19,func2=2"

Commit message: rev3
Parts:
- J4: footprint Pin_Headers:Pin_Header_Straight_1x07_Pitch2.54mm -> Pin_Headers:Pin_Header_Straight_1x08_Pitch2.54mm
- J5: footprint Connectors:BARREL_JACK -> _LaurentPerso:BARREL_JACK
- moved REF*** 0.81 mm to (40.4, 35.0)
Routing:
- net GND: track 121.2 -> 135.0 mm
- net /IO25: track 0.00 -> 10.9 mm
- net /B4: track 37.8 -> 40.4 mm
- net /IO26: track 17.7 -> 20.2 mm
- net /B5: track 40.2 -> 42.1 mm
- net /G2: track 30.1 -> 31.5 mm
- net /G6: track 38.6 -> 39.6 mm
- net /RPWM: track 35.8 -> 36.8 mm
- net /G3: track 30.9 -> 31.7 mm
Other:
- board text added: "Desingned by Laurent Le Goff (2017) http://github.com/llegoff/VGA_Zero Use dtoverlay vga565 with parameter dpi_output_format=0x13 For Audio dtoverlay=pwm-2chan,pin=18,func=2,pin2=19,func2=2"
- board text added: "IO25"
- board text removed: "Desingned by Laurent Le Goff (2017) http://github.com/llegoff/VGA_Zero Use dtoverlay dpi24 with parameter dpi_output_format=0x13 For Audio & SPI, remake dpi24.dtbo without pin GPIO 9 10 11 18 19 25 26 27 dtoverlay=pwm-2chan,pin=18,func=2,pin2=19,func2=2"

Commit message: rev3
Parts:
- added J6: BARREL_JACK, _LaurentPerso:DC002_3.5x1.1, F.Cu at (31.0, 20.0)
- moved J5 0.25 mm to (31.0, 30.2)
Changed lines of the file:
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@@
     (tracks 440)
     (zones 0)
-    (modules 33)
+    (modules 34)
     (nets 47)
   )
@@
   )
   (module _LaurentPerso:BARREL_JACK (layer F.Cu)
-    (at 31 30 270)
+    (at 31 30.25 270)
     (descr "DC Barrel Jack")
     (tags "Power Jack")
-    (fp_text reference J5 (at -9.05 3 180) (layer F.SilkS)
+    (fp_text reference J5 (at -9.05 3.5 180) (layer F.SilkS)
       (effects (font (size 1 1) (thickness 0.15)))
     )
@@
     )
   )
+  (module _LaurentPerso:DC002_3.5x1.1 (layer F.Cu)
+    (at 31 20 270)
+    (fp_text reference J6 (at 1.25 -1.5) (layer F.SilkS)
+      (effects (font (size 1 1) (thickness 0.15)))
+    )
+    (fp_text value BARREL_JACK (at 4 -3.5 270) (layer F.Fab)
+      (effects (font (size 1 1) (thickness 0.15)))
+    )
+    (fp_line (start 0 -2.5) (end 9.1 -2.5) (layer F.SilkS) (width 0.15))
+    (fp_line (start 0 2.5) (end 9.1 2.5) (layer F.SilkS) (width 0.15))
+    (fp_line (start 9.1 2.5) (end 9.1 -2.5) (layer F.SilkS) (width 0.15))
+    (fp_line (start 0 -2.5) (end -2 -2.5) (layer F.Fab) (width 0.15))
+    (fp_line (start -2 -2.5) (end -2 2.5) (layer F.Fab) (width 0.15))
+    (fp_line (start -2 2.5) (end 0 2.5) (layer F.Fab) (width 0.15))
+    (fp_line (start 0 -2.5) (end 0 2.5) (layer F.Fab) (width 0.15))
+    (pad 2 thru_hole oval (at 4 0 270) (size 1.6 2) (drill oval 0.8 1.2) (layers *.Cu *.Mask)
+      (net 14 GND))
+    (pad 3 thru_hole oval (at 6.3 2.8 270) (size 1.6 2) (drill oval 0.8 1.2) (layers *.Cu *.Mask)
+      (net 14 GND))
+    (pad 1 thru_hole oval (at 8.9 0 270) (size 1.6 2) (drill oval 0.8 1.2) (layers *.Cu *.Mask)
+      (net 46 /5V))
+  )
   (gr_text IO25 (at 43.65 39.4 90) (layer F.SilkS)

Commit message: Kicad v5.0.2 lib
Parts:
- removed REF***: KiCad-Logo2_6mm_SilkScreen, Symbols:KiCad-Logo2_6mm_SilkScreen
- removed REF***: OSHW-Logo2_7.3x6mm_SilkScreen, Symbols:OSHW-Logo2_7.3x6mm_SilkScreen
- J5: footprint _LaurentPerso:BARREL_JACK -> Connectors:BARREL_JACK
Routing:
- net Net-(C4-Pad2): track 14.9 -> 24.0 mm
- net Net-(C2-Pad2): track 25.0 -> 22.3 mm
